Commit message: first version

File: my_robot.xacro (robot description, xacro)
@@ -2,13 +2,13 @@
 <robot name="my_robot" xmlns:xacro="http://www.ros.org/wiki/xacro">
 <xacro:include filename="$(find my_robot)/urdf/my_robot.gazebo" />
-<link name="robot_footprint"></link>
 <gazebo reference="left_wheel">
-    <material>Gazebo/Yellow</material>
+    <material>Gazebo/Pink</material>
 </gazebo>
 <gazebo reference="right_wheel">
+    <material>Gazebo/Pink</material>
+</gazebo>
+  <link name="robot_footprint"></link>
+<gazebo reference="chassis">
     <material>Gazebo/Yellow</material>
-</gazebo>
-<gazebo reference="chassis">
-    <material>Gazebo/Red</material>
 </gazebo>
 <gazebo reference="hokuyo">
